Commit message: setup gazebo,next repair launch file

File: src/sentinel_publisher/description/imu.xacro (robot description, xacro)
@@ -3,23 +3,31 @@
     <joint name="imu_joint" type="fixed">
         <parent link="chassis"/>
-        <child link="imu_frame"/>
-	<origin xyz="0.0 0 0.155" rpy="0 0 0"/>
+        <child link="imu_link"/>
+        <origin xyz="0.0 0 0.155" rpy="0 0 0"/>
     </joint>
-    <link name="imu_frame">
-    <visual>
-        <origin xyz="0 0 0" rpy="0 0 1.5708"/>
-        <geometry>
-            <box size="0.01 0.01 0.005"/>
-        </geometry>
-        <material name="blue"/>
-    </visual>
-    <collision>
-        <geometry>
-        <cylinder radius="0.05" length="0.04"/>
-        </geometry>
-    </collision>
-    <xacro:inertial_cylinder mass="0.001" length="0.04" radius="0.05">
-        <origin xyz="0 0 0" rpy="0 0 0"/>
-    </xacro:inertial_cylinder>
+    <link name="imu_link">
+        <visual>
+            <origin xyz="0 0 0" rpy="0 0 1.5708"/>
+            <geometry>
+                <box size="0.01 0.01 0.005"/>
+            </geometry>
+            <material name="blue"/>
+        </visual>
+        <collision>
+            <geometry>
+                <cylinder radius="0.05" length="0.04"/>
+            </geometry>
+        </collision>
+        <xacro:inertial_cylinder mass="0.001" length="0.04" radius="0.05">
+            <origin xyz="0 0 0" rpy="0 0 0"/>
+        </xacro:inertial_cylinder>
     </link>
+    <gazebo reference="imu_link">
+        <sensor name="imu_sensor" type="imu">
+            <always_on>true</always_on>
+            <update_rate>100</update_rate>
+            <topic>imu</topic>
+            <gz_frame_id>imu_link</gz_frame_id>
+        </sensor>
+    </gazebo>
 </robot>

File: src/sentinel_publisher/description/lidar.xacro (robot description, xacro)
@@ -1,25 +1,56 @@
 <?xml version="1.0"?>
-<robot xmlns:xacro="http://www.ros.org/wiki/xacro" >
-    <joint name="laser_joint" type="fixed">
-        <parent link="chassis"/>
-        <child link="laser_frame"/>
-	<origin xyz="0.113 0 0.15" rpy="0 0 0"/>
-    </joint>
-    <link name="laser_frame">
-    <visual>
-        <origin xyz="0 0 0" rpy="0 0 1.5708"/>
-        <geometry>
-            <mesh filename="package://sentinel_publisher/meshes/rplidar.stl" scale="0.001 0.001 0.001"/>
-        </geometry>
-        <material name="red"/>
-    </visual>
-    <collision>
-        <geometry>
-        <cylinder radius="0.05" length="0.04"/>
-        </geometry>
-    </collision>
-    <xacro:inertial_cylinder mass="0.001" length="0.04" radius="0.05">
-        <origin xyz="0 0 0" rpy="0 0 0"/>
-    </xacro:inertial_cylinder>
-    </link>
+<robot xmlns:xacro="http://www.ros.org/wiki/xacro">
+  <xacro:include filename="inertial_macros.xacro"/>
+  <joint name="laser_joint" type="fixed">
+    <parent link="chassis"/>
+    <child link="laser_frame"/>
+    <origin xyz="0.113 0 0.15" rpy="0 0 0"/>
+  </joint>
+  <link name="laser_frame">
+  <visual>
+    <geometry>
+      <mesh filename="package://sentinel_publisher/meshes/rplidar.stl" scale="0.001 0.001 0.001"/>
+    </geometry>
+    <material name="red"/>
+  </visual>
+  <collision>
+    <geometry>
+      <cylinder radius="0.05" length="0.04"/>
+    </geometry>
+  </collision>
+  <xacro:inertial_cylinder mass="0.001" length="0.04" radius="0.05">
+    <origin xyz="0 0 0" rpy="0 0 0"/>
+  </xacro:inertial_cylinder>
+  </link>
+  <!-- Gazebo Harmonic native lidar -->
+  <gazebo reference="laser_frame">
+      <sensor name="gpu_lidar" type="gpu_lidar">
+      <pose relative_to="laser_frame">0 0 0.03 0 0 0</pose>
+      <topic>scan</topic>
+      <update_rate>10</update_rate>
+        <lidar>
+          <scan>
+            <horizontal>
+              <samples>720</samples>
+              <resolution>1</resolution>
+              <min_angle>-3.1459</min_angle>
+              <max_angle>3.1459</max_angle>
+            </horizontal>
+          </scan>
+          <range>
+            <min>0.01</min>
+            <max>12</max>
+            <resolution>0.005</resolution>
+          </range>
+          <noise>
+            <type>gaussian</type>
+            <mean>0</mean>
+            <stddev>0.001</stddev>
+          </noise>
+        </lidar>
+        <gz_frame_id>laser_frame</gz_frame_id>
+        <visualize>true</visualize>
+        <always_on>1</always_on>
+      </sensor>
+  </gazebo>
 </robot>

File: src/sentinel_publisher/description/robot_core.xacro (robot description, xacro)
@@ -47,5 +47,5 @@
             <origin xyz="0.0 0.0 0.1" rpy="0.0 0.0 0.0"/>
             <geometry>
-                <box size="0.426 0.30 0.03"/>
+                <box size="0.426 0.30 0.1"/>
             </geometry>
             <material name="white"/>

File: src/sentinel_publisher/description/ros2_control.xacro (robot description, xacro)
@@ -1,31 +1,29 @@
 <?xml version="1.0"?>
 <robot xmlns:xacro="http://www.ros.org/wiki/xacro">
-    <ros2_control name="RealRobot" type="system">
-      <hardware>
-        <plugin>diffdrive_arduino/DiffDriveArduinoHardware</plugin>
-          <param name="left_wheel_name">left_wheel_joint</param>
-          <param name="right_wheel_name">right_wheel_joint</param>
-          <param name="loop_rate">30</param>
-          <param name="device">/dev/arduino_nano</param>
-          <param name="baud_rate">57600</param>
-          <param name="timeout_ms">3000</param>
-          <param name="enc_counts_per_rev">2000</param>
-      </hardware>
-      <joint name="left_wheel_joint">
-        <command_interface name="velocity">
-          <param name="min">-10</param>
-          <param name="max">10</param>
-        </command_interface>
-        <state_interface name="position"/>
-        <state_interface name="velocity"/>
-      </joint>
-      <joint name="right_wheel_joint">
-        <command_interface name="velocity">
-          <param name="min">-10</param>
-          <param name="max">10</param>
-        </command_interface>
-        <state_interface name="position"/>
-        <state_interface name="velocity"/>
-      </joint>
-    </ros2_control>
+  <ros2_control name="GazeboSimSystem" type="system">
+    <hardware>
+      <plugin>gz_ros2_control/GazeboSimSystem</plugin>
+    </hardware>
+    <joint name="left_wheel_joint">
+      <command_interface name="velocity">
+        <param name="min">-10</param>
+        <param name="max">10</param>
+      </command_interface>
+      <state_interface name="position"/>
+      <state_interface name="velocity"/>
+    </joint>
+    <joint name="right_wheel_joint">
+      <command_interface name="velocity">
+        <param name="min">-10</param>
+        <param name="max">10</param>
+      </command_interface>
+      <state_interface name="position"/>
+      <state_interface name="velocity"/>
+    </joint>
+  </ros2_control>
+  <gazebo>
+    <plugin filename="gz_ros2_control-system" name="gz_ros2_control::GazeboSimROS2ControlPlugin">
+      <parameters>$(find sentinel_publisher)/config/my_controllers.yaml</parameters>
+    </plugin>
+  </gazebo>
 </robot>

Commit message: update25may

File: src/sentinel_publisher/description/imu.xacro (robot description, xacro)
@@ -2,7 +2,7 @@
 <robot xmlns:xacro="http://www.ros.org/wiki/xacro" >
     <joint name="imu_joint" type="fixed">
+        <origin xyz="0.0 0 0.155" rpy="0 0 0"/>
         <parent link="chassis"/>
         <child link="imu_link"/>
-        <origin xyz="0.0 0 0.155" rpy="0 0 0"/>
     </joint>
     <link name="imu_link">
@@ -24,9 +24,11 @@
     </link>
     <gazebo reference="imu_link">
-        <sensor name="imu_sensor" type="imu">
-            <always_on>true</always_on>
-            <update_rate>100</update_rate>
-            <topic>imu</topic>
-            <gz_frame_id>imu_link</gz_frame_id>
+        <sensor name="imu" type="imu">
+        <always_on>1</always_on>
+        <update_rate>50</update_rate>
+        <visualize>true</visualize>
+        <topic>imu</topic>
+        <enable_metrics>true</enable_metrics>
+        <gz_frame_id>imu_link</gz_frame_id>
         </sensor>
     </gazebo>
