Commit message: update ros2 integration

File: src/diffdrive_arduino/description/ros2_control/diffbot.ros2_control.xacro (robot description, xacro)
@@ -12,6 +12,6 @@
         <param name="timeout_ms">1000</param>
         <param name="enc_counts_per_rev">3436</param>
-        <param name="pid_p">20</param>
-        <param name="pid_d">12</param>
+        <param name="pid_p">70</param>
+        <param name="pid_d">110</param>
         <param name="pid_i">0</param>
         <param name="pid_o">50</param>

File: src/sentinel_publisher/description/lidar.xacro (robot description, xacro)
@@ -5,5 +5,6 @@
     <parent link="chassis"/>
     <child link="laser_frame"/>
-    <origin xyz="0.113 0 0.15" rpy="0 0 0"/>
+    <!-- <origin xyz="0.113 0 0.15" rpy="0 0 1.2008"/>  dreame lds lidar -->
+    <origin xyz="0.113 0 0.15" rpy="0 0 0"/> <!-- A2 -->
   </joint>
   <link name="laser_frame">

File: src/sentinel_publisher/description/ros2_control.xacro (robot description, xacro)
@@ -6,9 +6,13 @@
         <param name="left_wheel_name">left_wheel_joint</param>
         <param name="right_wheel_name">right_wheel_joint</param>
-        <param name="loop_rate">30</param>
+        <param name="loop_rate">20</param>
         <param name="device">/dev/ttySTM32</param>
         <param name="baud_rate">115200</param>
-        <param name="timeout_ms">3000</param>
+        <param name="timeout_ms">1000</param>
         <param name="enc_counts_per_rev">595</param>
+        <param name="pid_p">70</param>
+        <param name="pid_d">110</param>
+        <param name="pid_i">0</param>
+        <param name="pid_o">50</param>
     </hardware>
     <joint name="left_wheel_joint">
